File: hardware/fencing_scoring_box/fencing_scoring_box.kicad_pcb (KiCad board)
At the start: 2 copper layers, 100 x 70 mm, 38 parts, among them J1 LED_Matrix, J10 Grn LEDs, J13 Grn, J14 Red, J3 Conn_01x01, J4 Red LEDs, J7 Mode_LEDs, SW1 SW_Push

Commit message: Pin changes to arduino code and renaming pcb design
Changed the pins to be compatibe with the new PCB design for an arduino
nano
Parts:
- H1: value Piste Connetor -> Piste Gnd
- SW1: value SW_Push -> Weapon Select
Changed lines of the file:
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@@
 			(plot_on_all_layers_selection 0x0001000_00000000)
 			(disableapertmacros no)
-			(usegerberextensions yes)
+			(usegerberextensions no)
 			(usegerberattributes no)
 			(usegerberadvancedattributes no)
@@
 			(psa4output no)
 			(plotreference yes)
-			(plotvalue no)
+			(plotvalue yes)
 			(plotfptext yes)
 			(plotinvisibletext no)
@@
 			)
 		)
-		(property "Value" "SW_Push"
+		(property "Value" "Weapon Select"
 			(at 9.75 2.05 180)
 			(layer "F.SilkS")
@@
 			(at -3.13 0 0)
 			(unlocked yes)
-			(layer "F.Fab")
+			(layer "F.SilkS")
 			(effects
 				(font
@@
 			(at -3.18 0 0)
 			(unlocked yes)
-			(layer "F.Fab")
+			(layer "F.SilkS")
 			(effects
 				(font
@@
 			)
 		)
-		(property "Value" "Piste Connetor"
-			(at 0.25 -5 0)
+		(property "Value" "Piste Gnd"
+			(at -8.5 3.5 0)
 			(unlocked yes)
-			(layer "F.Fab")
-			(hide yes)
+			(layer "F.SilkS")
 			(effects
 				(font
