File: designs/epee_buzz_box/hardware/epee_buzz_box/epee_buzz_box.kicad_sch (KiCad schematic)
At the start: 13 parts, among them J13 Grn

Commit message: Adding LED to the schematic
Parts:
- added D1: LED, symbol Device:LED
- added R1: 220, my_library:resistor_THT_and_0805, symbol fencing_scoring-box-rescue:R_Small-RESCUE-fencing_scoring_box
Connections:
- net GND: now also R1.1
- net Grn_OnT_LED renamed OnT_LED
- net OnT_LED: now also D1.2 (A)
- new net: D1.1 (K), R1.2
