File: designs/wired_scoring_box/hardware/fencing_scoring_box/fencing_scoring_box.kicad_pcb (KiCad board)
At the start: 2 copper layers, 100 x 70 mm, 38 parts, among them J1 LED_Matrix, J10 Grn LEDs, J13 Grn, J14 Red, J3 Conn_01x01, J4 Red LEDs, J7 Mode_LEDs, SW1 Weapon Select

Commit message: PCB Version 5 firmware and pcb updates
1. Updated the firmware to support only one matrix of 64 LEDs
2. Updated the PCB design error found when assembling the PCB
    - Turns out the Arduino Nano A6 and A7 pins cant be used as digital
      and now the display runs off pin 13 rather than pin A6
    - Corrected some pin names on the silkscreen
Still need to increase the hole size for the button to protrude through the
display board
Parts:
- H1: value Piste Gnd -> Piste Connetor
- moved J7 0.50 mm to (147.2, 65.9)
Connections:
- A1 pad 16: unconnected-(A1-D13-Pad16) -> display1
- A1 pad 25: display1 -> unconnected-(A1-A6-Pad25)
Routing:
- net display1: track 23.2 -> 46.1 mm, vias 0 -> 1
