File: designs/wired_scoring_box/hardware/fencing_scoring_box/fencing_scoring_box.kicad_sch (KiCad schematic)
At the start: 50 parts, among them J1 LED_Matrix, J10 Grn LEDs, J13 Grn, J14 Red, J3 Conn_01x01, J4 Red LEDs, J5 Button, J7 Mode_LEDs, SW1 SW_Push

Commit message: PCB Version 5 firmware and pcb updates
1. Updated the firmware to support only one matrix of 64 LEDs
2. Updated the PCB design error found when assembling the PCB
    - Turns out the Arduino Nano A6 and A7 pins cant be used as digital
      and now the display runs off pin 13 rather than pin A6
    - Corrected some pin names on the silkscreen
Still need to increase the hole size for the button to protrude through the
display board
Parts:
- D1, D2, D3, D4, D5, D6: value D_Zener -> D_Zen
- SW1: value SW_Push -> Weapon Select
Connections:
- net display1: now also A1.16 (D13); no longer A1.25 (A6)
Changed lines of the file:
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@@
 	)
 	(no_connect
-		(at 123.19 82.55)
+		(at 153.67 80.01)
 	)
 	(no_connect
@@
 	(wire
 		(pts
-			(xy 153.67 80.01) (xy 157.48 80.01)
-		)
-		(stroke
-			(width 0)
-			(type default)
-		)
-	)
-	(wire
-		(pts
 			(xy 261.62 105.41) (xy 261.62 102.87)
 		)
@@
 		)
 	)
+	(global_label "display1"
+		(shape input)
+		(at 123.19 82.55 180)
+		(effects
+			(font
+				(size 1.524 1.524)
+			)
+			(justify right)
+		)
+		(property "Intersheetrefs" "${INTERSHEET_REFS}"
+			(at 123.19 82.55 0)
+			(effects
+				(font
+					(size 1.27 1.27)
+				)
+				(hide yes)
+			)
+		)
+	)
 	(global_label "Red_A_out"
 		(shape input)
@@
 		)
 	)
-	(global_label "display1"
-		(shape input)
-		(at 157.48 80.01 0)
-		(effects
-			(font
-				(size 1.524 1.524)
-			)
-			(justify left)
-		)
-		(property "Intersheetrefs" "${INTERSHEET_REFS}"
-			(at 157.48 80.01 0)
-			(effects
-				(font
-					(size 1.27 1.27)
-				)
-				(hide yes)
-			)
-		)
-	)
 	(global_label "Red_OffT_LED"
 		(shape input)
@@
 			)
 		)
-		(property "Value" "D_Zener"
+		(property "Value" "D_Zen"
 			(at 196.85 78.74 0)
 			(effects
@@
 			)
 		)
-		(property "Value" "D_Zener"
+		(property "Value" "D_Zen"
 			(at 250.19 78.74 0)
 			(effects
@@
 			)
 		)
-		(property "Value" "D_Zener"
+		(property "Value" "D_Zen"
 			(at 196.85 100.33 0)
 			(effects
@@
 			)
 		)
-		(property "Value" "D_Zener"
+		(property "Value" "D_Zen"
 			(at 250.19 100.33 0)
 			(effects
@@
 			)
 		)
-		(property "Value" "D_Zener"
+		(property "Value" "D_Zen"
 			(at 198.12 129.54 0)
 			(effects
@@
 			)
 		)
-		(property "Value" "D_Zener"
+		(property "Value" "D_Zen"
 			(at 251.46 129.54 0)
 			(effects
@@
 			)
 		)
-		(property "Value" "SW_Push"
+		(property "Value" "Weapon Select"
 			(at 68.326 81.28 0)
 			(effects
