File: designs/wired_scoring_box/hardware/fencing_scoring_box_led_matrix/fencing_scoring_box_led_matrix.kicad_pcb (KiCad board)
At the start: 2 copper layers, 100 x 70 mm, 11 parts, among them J2 Conn_01x05_Pin

Commit message: Updates to the matrix display board
Updated the ws2812b 4x4 matrix footprint and symbol
Increased the size of the buzzer and button holes
Routing:
- net GND: track 138.4 -> 104.9 mm, vias 0 -> 12
- net 5V: track 0.00 -> 10.0 mm
- net Net-(U3-Output): track 5.50 -> 5.00 mm
- net Net-(U1-Output): track 5.50 -> 5.00 mm
Other:
- outline, holes or cut-outs redrawn
