File: designs/wired_scoring_box/hardware/fencing_scoring_box_led_matrix/fencing_scoring_box_led_matrix.kicad_sch (KiCad schematic)
At the start: 9 parts, among them J2 Conn_01x05_Pin

Commit message: Updates to the matrix display board
Updated the ws2812b 4x4 matrix footprint and symbol
Increased the size of the buzzer and button holes
Connections:
- net GND: no longer U1.9 (GND), U2.9 (GND), U3.9 (GND), U4.9 (GND)
Changed lines of the file:
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@@
-	)
-	(junction
-		(at 184.15 83.82)
-		(diameter 0)
-		(color 0 0 0 0)
-	)
-	(junction
-		(at 152.4 83.82)
-		(diameter 0)
-		(color 0 0 0 0)
 	)
 	(junction
@@
 	)
 	(junction
-		(at 120.65 83.82)
-		(diameter 0)
-		(color 0 0 0 0)
-	)
-	(junction
 		(at 176.53 83.82)
 		(diameter 0)
@@
 		(color 0 0 0 0)
 	)
-	(junction
-		(at 88.9 83.82)
-		(diameter 0)
-		(color 0 0 0 0)
-	)
 	(no_connect
 		(at 194.31 74.93)
@@
 	(wire
 		(pts
-			(xy 152.4 83.82) (xy 154.94 83.82)
-		)
-		(stroke
-			(width 0)
-			(type default)
-		)
-	)
-	(wire
-		(pts
 			(xy 83.82 63.5) (xy 83.82 67.31)
 		)
@@
 	(wire
 		(pts
-			(xy 184.15 83.82) (xy 186.69 83.82)
-		)
-		(stroke
-			(width 0)
-			(type default)
-		)
-	)
-	(wire
-		(pts
 			(xy 99.06 74.93) (xy 105.41 74.93)
 		)
@@
 	(wire
 		(pts
-			(xy 120.65 83.82) (xy 123.19 83.82)
-		)
-		(stroke
-			(width 0)
-			(type default)
-		)
-	)
-	(wire
-		(pts
 			(xy 64.77 69.85) (xy 64.77 72.39)
-		)
-		(stroke
-			(width 0)
-			(type default)
-		)
-	)
-	(wire
-		(pts
-			(xy 88.9 83.82) (xy 91.44 83.82)
 		)
 		(stroke
@@
 			)
 		)
-		(pin "9"
-		)
 		(pin "8"
 		)
@@
 	)
 	(symbol
+		(lib_name "WS2812b_4x4_Matrix_1")
 		(lib_id "my_library:WS2812b_4x4_Matrix")
 		(at 86.36 25.4 0)
@@
 			)
 		)
-		(pin "9"
-		)
 		(pin "8"
 		)
@@
 	)
 	(symbol
+		(lib_name "WS2812b_4x4_Matrix_3")
 		(lib_id "my_library:WS2812b_4x4_Matrix")
 		(at 149.86 25.4 0)
@@
 			)
 		)
-		(pin "9"
-		)
 		(pin "8"
 		)
@@
 	)
 	(symbol
+		(lib_name "WS2812b_4x4_Matrix_2")
 		(lib_id "my_library:WS2812b_4x4_Matrix")
 		(at 118.11 25.4 0)
@@
 			)
 		)
-		(pin "9"
-		)
 		(pin "8"
